File: Celestron-WiFi.kicad_pcb (KiCad board)
At the start: 4 copper layers, 28.4 x 60.5 mm, 23 parts, among them J1 GPS, J2 6P6C, Q1 UMH3N, SW1 RESET, SW2 SW_DIP_x04, U1 LM2672M-3.3, U2 ESP32-WROOM-32U, U3 74LVC125

Commit message: routing changes
Parts:
- C1: footprint Capacitor_Tantalum_SMD:CP_EIA-2012-12_Kemet-R -> Capacitor_Tantalum_SMD:CP_EIA-7343-43_Kemet-X
- C5: footprint Capacitor_Tantalum_SMD:CP_EIA-2012-12_Kemet-R -> Capacitor_Tantalum_SMD:CP_EIA-3216-18_Kemet-A
- C6: footprint Capacitor_SMD:C_0603_1608Metric -> Capacitor_SMD:C_0805_2012Metric
- R3, R4: value 50K -> 49.9K
- U3: value 74LVC125 -> 74HC125; footprint Package_SO:SOIC-14_3.9x8.7mm_P1.27mm -> Package_SO:TSSOP-14_4.4x5mm_P0.65mm
- moved R4 18.8 mm to (135.6, 110.7)
- moved R1 11.9 mm to (114.9, 78.2), turned to -90 degrees
- moved C3 11.9 mm to (112.8, 78.2), turned to -90 degrees
- moved C1 10.2 mm to (115.2, 109.2)
- moved D1 0.52 mm to (123.1, 97.5)
- moved R3 0.51 mm to (135.6, 106.4)
Routing:
- net +12V: track 13.6 -> 24.7 mm
- net IO33: track 43.3 -> 34.2 mm
- net IO32: track 40.0 -> 32.9 mm
- net EN: track 32.3 -> 29.2 mm
- net /TX: track 44.6 -> 41.6 mm
- net RXD0: track 32.9 -> 31.1 mm
- net /BUSY: track 38.1 -> 36.5 mm
- net TXD0: track 27.7 -> 29.2 mm
- net GND: track 36.2 -> 34.9 mm, vias 20 -> 36
- net W_RST: track 22.1 -> 23.2 mm
Other:
- rule pad_to_mask_clearance: 0 -> 0.0508
- board text added: "1"
- board text added: "1. WiFi Enable 2. Evo Mount WiFi Enable 3. WiFi Reset 4. WiFi Mode (Direct/Access)"
- board text added: "2"
- board text added: "3"
- board text added: "4"
- board text added: "GPS"
- board text added: "PWR"
- board text removed: "1. WiFi Enable 2. Evo Mount WiFi Enable 3. WiFi Reset 4. WiFi Mode"

Commit message: schematic fixes
Parts:
- U2: value ESP32-WROOM-32U -> ESP32-WROOM-32D; footprint RF_Module:ESP32-WROOM-32U -> RF_Module:ESP32-WROOM-32
- moved C1 0.13 mm to (115.3, 109.2)
- renumbered J2 to J1, J1 to J2
Connections:
- net /BUSY renamed Net-(J1-Pad6)
- U2 pad 9: IO33 -> RTS
- U3 pad 11: IO33 -> RTS
Routing:
- net RTS: track 2.17 -> 37.7 mm, vias 0 -> 3
- net IO33: track 34.2 -> 0.00 mm, vias 2 -> 0
- net EN: track 29.2 -> 28.6 mm
- net GND: vias 36 -> 37
Other:
- board size 28.4 x 60.5 mm -> 28.4 x 66.3 mm
