File: Celestron-WiFi.kicad_sch (KiCad schematic)
At the start: 22 parts, among them J1 GPS, J2 6P6C, Q1 UMH3N, SW1 RESET, SW2 SW_DIP_x04, U1 LM2672M-3.3, U2 ESP32-WROOM-32U, U3 74LVC125

Commit message: routing changes
Parts:
- C1: footprint Capacitor_Tantalum_SMD:CP_EIA-2012-12_Kemet-R -> Capacitor_Tantalum_SMD:CP_EIA-7343-43_Kemet-X; MPN (none) -> T491X107M025AT
- C5: footprint Capacitor_Tantalum_SMD:CP_EIA-2012-12_Kemet-R -> Capacitor_Tantalum_SMD:CP_EIA-3216-18_Kemet-A; MPN (none) -> T491A686K006AT
- C6: footprint Capacitor_SMD:C_0603_1608Metric -> Capacitor_SMD:C_0805_2012Metric; MPN (none) -> C0805C226M8PACTU
- D1: MPN (none) -> PD3S230LQ-7
- R1: MPN (none) -> CR0603-FX-1000ELF
- R3, R4: value 50K -> 49.9K; MPN (none) -> CR0603-FX-4992ELF
- SW2: MPN (none) -> 219-4MS
- U1: MPN (none) -> LM2672M-3.3/NOPB
- U3: value 74LVC125 -> 74HC125; footprint Package_SO:SOIC-14_3.9x8.7mm_P1.27mm -> Package_SO:TSSOP-14_4.4x5mm_P0.65mm
Changed lines of the file:
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@@
+      (effects (font (size 1.27 1.27)) hide)
+    )
+    (property "MPN" "LM2672M-3.3/NOPB" (id 4) (at 53.34 168.91 0)
       (effects (font (size 1.27 1.27)) hide)
     )
@@
     (in_bom yes) (on_board yes) (fields_autoplaced)
     (property "Reference" "U3" (id 0) (at 200.66 19.05 0))
-    (property "Value" "74LVC125" (id 1) (at 200.66 21.59 0))
-    (property "Footprint" "Package_SO:SOIC-14_3.9x8.7mm_P1.27mm" (id 2) (at 200.66 27.94 0)
+    (property "Value" "74HC125" (id 1) (at 200.66 21.59 0))
+    (property "Footprint" "Package_SO:TSSOP-14_4.4x5mm_P0.65mm" (id 2) (at 200.66 27.94 0)
       (effects (font (size 1.27 1.27)) hide)
     )
@@
       (effects (font (size 1.27 1.27)) hide)
     )
+    (property "MPN" "CR0603-FX-1000ELF" (id 4) (at 45.72 72.39 0)
+      (effects (font (size 1.27 1.27)) hide)
+    )
     (pin "1")
     (pin "2")
@@
       (effects (font (size 1.27 1.27)) (justify left))
     )
-    (property "Footprint" "Capacitor_SMD:C_0603_1608Metric" (id 2) (at 110.49 127 0)
+    (property "Footprint" "Capacitor_SMD:C_0805_2012Metric" (id 2) (at 110.49 127 0)
       (effects (font (size 1.27 1.27)) hide)
     )
     (property "Datasheet" "~" (id 3) (at 110.49 127 0)
+      (effects (font (size 1.27 1.27)) hide)
+    )
+    (property "MPN" "C0805C226M8PACTU" (id 4) (at 110.49 127 0)
       (effects (font (size 1.27 1.27)) hide)
     )
@@
       (effects (font (size 1.27 1.27)) (justify left))
     )
-    (property "Value" "74LVC125" (id 1) (at 157.48 172.7199 0)
-      (effects (font (size 1.27 1.27)) (justify left))
-    )
-    (property "Footprint" "Package_SO:SOIC-14_3.9x8.7mm_P1.27mm" (id 2) (at 151.13 171.45 0)
+    (property "Value" "74HC125" (id 1) (at 157.48 172.7199 0)
+      (effects (font (size 1.27 1.27)) (justify left))
+    )
+    (property "Footprint" "Package_SO:TSSOP-14_4.4x5mm_P0.65mm" (id 2) (at 151.13 171.45 0)
       (effects (font (size 1.27 1.27)) hide)
     )
@@
     (in_bom yes) (on_board yes) (fields_autoplaced)
     (property "Reference" "U3" (id 0) (at 200.66 87.63 0))
-    (property "Value" "74LVC125" (id 1) (at 200.66 90.17 0))
-    (property "Footprint" "Package_SO:SOIC-14_3.9x8.7mm_P1.27mm" (id 2) (at 200.66 96.52 0)
+    (property "Value" "74HC125" (id 1) (at 200.66 90.17 0))
+    (property "Footprint" "Package_SO:TSSOP-14_4.4x5mm_P0.65mm" (id 2) (at 200.66 96.52 0)
       (effects (font (size 1.27 1.27)) hide)
     )
@@
       (effects (font (size 1.27 1.27)) (justify left))
     )
-    (property "Footprint" "Capacitor_Tantalum_SMD:CP_EIA-2012-12_Kemet-R" (id 2) (at 31.75 177.8 0)
-      (effects (font (size 1.27 1.27)) hide)
-    )
-    (property "Datasheet" "~" (id 3) (at 31.75 177.8 0)
+    (property "Footprint" "Capacitor_Tantalum_SMD:CP_EIA-7343-43_Kemet-X" (id 2) (at 31.75 177.8 0)
+      (effects (font (size 1.27 1.27)) hide)
+    )
+    (property "Datasheet" "https://www.mouser.com/datasheet/2/212/1/KEM_T2005_T491-1093550.pdf" (id 3) (at 31.75 177.8 0)
+      (effects (font (size 1.27 1.27)) hide)
+    )
+    (property "MPN" "T491X107M025AT" (id 4) (at 31.75 177.8 0)
       (effects (font (size 1.27 1.27)) hide)
     )
@@
     (in_bom yes) (on_board yes) (fields_autoplaced)
     (property "Reference" "U3" (id 0) (at 200.66 40.64 0))
-    (property "Value" "74LVC125" (id 1) (at 200.66 43.18 0))
-    (property "Footprint" "Package_SO:SOIC-14_3.9x8.7mm_P1.27mm" (id 2) (at 200.66 49.53 0)
+    (property "Value" "74HC125" (id 1) (at 200.66 43.18 0))
+    (property "Footprint" "Package_SO:TSSOP-14_4.4x5mm_P0.65mm" (id 2) (at 200.66 49.53 0)
       (effects (font (size 1.27 1.27)) hide)
     )
@@
   (symbol (lib_id "Device:R_Small") (at 237.49 44.45 0) (mirror y) (unit 1)
     (in_bom yes) (on_board yes)
-    (property "Reference" "R4" (id 0) (at 242.57 44.45 0)
-      (effects (font (size 1.27 1.27)) (justify left))
-    )
-    (property "Value" "50K" (id 1) (at 242.57 46.99 0)
+    (property "Reference" "R4" (id 0) (at 241.3 44.45 0)
+      (effects (font (size 1.27 1.27)) (justify left))
+    )
+    (property "Value" "49.9K" (id 1) (at 243.84 46.99 0)
       (effects (font (size 1.27 1.27)) (justify left))
     )
@@
       (effects (font (size 1.27 1.27)) hide)
     )
-    (property "Datasheet" "~" (id 3) (at 237.49 44.45 0)
+    (property "Datasheet" "https://www.mouser.com/datasheet/2/54/crxxxxx-1858361.pdf" (id 3) (at 237.49 44.45 0)
+      (effects (font (size 1.27 1.27)) hide)
+    )
+    (property "MPN" "CR0603-FX-4992ELF" (id 4) (at 237.49 44.45 0)
       (effects (font (size 1.27 1.27)) hide)
     )
@@
     (in_bom yes) (on_board yes) (fields_autoplaced)
     (property "Reference" "U3" (id 0) (at 199.39 63.5 0))
-    (property "Value" "74LVC125" (id 1) (at 199.39 66.04 0))
-    (property "Footprint" "Package_SO:SOIC-14_3.9x8.7mm_P1.27mm" (id 2) (at 199.39 72.39 0)
+    (property "Value" "74HC125" (id 1) (at 199.39 66.04 0))
+    (property "Footprint" "Package_SO:TSSOP-14_4.4x5mm_P0.65mm" (id 2) (at 199.39 72.39 0)
       (effects (font (size 1.27 1.27)) hide)
     )
@@
       (effects (font (size 1.27 1.27)) hide)
     )
-    (property "Datasheet" "~" (id 3) (at 204.47 132.08 0)
+    (property "Datasheet" "https://www.mouser.com/datasheet/2/96/219-1144706.pdf" (id 3) (at 204.47 132.08 0)
+      (effects (font (size 1.27 1.27)) hide)
+    )
+    (property "MPN" "219-4MS" (id 4) (at 204.47 132.08 0)
       (effects (font (size 1.27 1.27)) hide)
     )
@@
       (effects (font (size 1.27 1.27)) (justify left))
     )
-    (property "Value" "50K" (id 1) (at 233.68 46.99 0)
+    (property "Value" "49.9K" (id 1) (at 233.68 46.99 0)
       (effects (font (size 1.27 1.27)) (justify left))
     )
@@
       (effects (font (size 1.27 1.27)) hide)
     )
-    (property "Datasheet" "~" (id 3) (at 234.95 44.45 0)
+    (property "Datasheet" "https://www.mouser.com/datasheet/2/54/crxxxxx-1858361.pdf" (id 3) (at 234.95 44.45 0)
+      (effects (font (size 1.27 1.27)) hide)
+    )
+    (property "MPN" "CR0603-FX-4992ELF" (id 4) (at 234.95 44.45 0)
       (effects (font (size 1.27 1.27)) hide)
     )
@@
       (effects (font (size 1.27 1.27)) hide)
     )
+    (property "MPN" "PD3S230LQ-7 " (id 4) (at 73.66 179.07 90)
+      (effects (font (size 1.27 1.27)) hide)
+    )
     (pin "1")
     (pin "2")
@@
       (effects (font (size 1.27 1.27)) (justify left))
     )
-    (property "Footprint" "Capacitor_Tantalum_SMD:CP_EIA-2012-12_Kemet-R" (id 2) (at 90.17 179.07 0)
-      (effects (font (size 1.27 1.27)) hide)
-    )
-    (property "Datasheet" "~" (id 3) (at 90.17 179.07 0)
+    (property "Footprint" "Capacitor_Tantalum_SMD:CP_EIA-3216-18_Kemet-A" (id 2) (at 90.17 179.07 0)
+      (effects (font (size 1.27 1.27)) hide)
+    )
+    (property "Datasheet" "https://www.mouser.com/datasheet/2/212/1/KEM_T2005_T491-1093550.pdf" (id 3) (at 90.17 179.07 0)
+      (effects (font (size 1.27 1.27)) hide)
+    )
+    (property "MPN" "T491A686K006AT" (id 4) (at 90.17 179.07 0)
       (effects (font (size 1.27 1.27)) hide)
     )
@@
     )
     (path "/7b2842dc-85a2-45a3-ab4f-abecb6110de2"
-      (reference "C1") (unit 1) (value "100uF") (footprint "Capacitor_Tantalum_SMD:CP_EIA-2012-12_Kemet-R")
+      (reference "C1") (unit 1) (value "100uF") (footprint "Capacitor_Tantalum_SMD:CP_EIA-7343-43_Kemet-X")
     )
     (path "/b90e5013-ee47-43b3-8670-9fa904e4538d"
@@
     )
     (path "/fdc82cbe-6ec7-4791-90d7-4f2a6e34d96d"
-      (reference "C5") (unit 1) (value "68uF") (footprint "Capacitor_Tantalum_SMD:CP_EIA-2012-12_Kemet-R")
+      (reference "C5") (unit 1) (value "68uF") (footprint "Capacitor_Tantalum_SMD:CP_EIA-3216-18_Kemet-A")
     )
     (path "/30cf36a5-3f53-4c68-8b80-384f94f56d03"
-      (reference "C6") (unit 1) (value "22uF") (footprint "Capacitor_SMD:C_0603_1608Metric")
+      (reference "C6") (unit 1) (value "22uF") (footprint "Capacitor_SMD:C_0805_2012Metric")
     )
     (path "/c15817ef-c68d-4d6b-93f4-89b65b251ef8"
@@
     )
     (path "/e6e468d8-2bb7-49d5-a4d0-fde0f6bbe8c6"
-      (reference "R3") (unit 1) (value "50K") (footprint "Resistor_SMD:R_0603_1608Metric")
+      (reference "R3") (unit 1) (value "49.9K") (footprint "Resistor_SMD:R_0603_1608Metric")
     )
     (path "/8313e187-c805-4927-8002-313a51839243"
-      (reference "R4") (unit 1) (value "50K") (footprint "Resistor_SMD:R_0603_1608Metric")
+      (reference "R4") (unit 1) (value "49.9K") (footprint "Resistor_SMD:R_0603_1608Metric")
     )
     (path "/6bbf7c3b-1a6b-43e6-98bb-6491d6bac7c8"
@@
     )
     (path "/824b4b92-8ae6-4ac2-b730-a8f5fa54180c"
-      (reference "U3") (unit 1) (value "74LVC125") (footprint "Package_SO:SOIC-14_3.9x8.7mm_P1.27mm")
+      (reference "U3") (unit 1) (value "74HC125") (footprint "Package_SO:TSSOP-14_4.4x5mm_P0.65mm")
     )
     (path "/281d6ad9-91e5-4114-8751-f23e609b642c"
-      (reference "U3") (unit 2) (value "74LVC125") (footprint "Package_SO:SOIC-14_3.9x8.7mm_P1.27mm")
+      (reference "U3") (unit 2) (value "74HC125") (footprint "Package_SO:TSSOP-14_4.4x5mm_P0.65mm")
     )
     (path "/79bf18db-f546-4b52-9e1a-426a24e165c6"
-      (reference "U3") (unit 3) (value "74LVC125") (footprint "Package_SO:SOIC-14_3.9x8.7mm_P1.27mm")
+      (reference "U3") (unit 3) (value "74HC125") (footprint "Package_SO:TSSOP-14_4.4x5mm_P0.65mm")
     )
     (path "/89fc496e-5b9b-4414-9b3a-38bef3e8aa03"
-      (reference "U3") (unit 4) (value "74LVC125") (footprint "Package_SO:SOIC-14_3.9x8.7mm_P1.27mm")
+      (reference "U3") (unit 4) (value "74HC125") (footprint "Package_SO:TSSOP-14_4.4x5mm_P0.65mm")
     )
     (path "/5145944b-e981-4bc0-be69-7b26bbe5a54c"
-      (reference "U3") (unit 5) (value "74LVC125") (footprint "Package_SO:SOIC-14_3.9x8.7mm_P1.27mm")
-    )
-  )
+      (reference "U3") (unit 5) (value "74HC125") (footprint "Package_SO:TSSOP-14_4.4x5mm_P0.65mm")
+    )
+  )

Commit message: schematic fixes
Parts:
- removed C1: 100uF, Capacitor_Tantalum_SMD:CP_EIA-7343-43_Kemet-X, symbol Device:CP_Small
- removed C5: 68uF, Capacitor_Tantalum_SMD:CP_EIA-3216-18_Kemet-A, symbol Device:CP_Small
- removed U2: ESP32-WROOM-32U, RF_Module:ESP32-WROOM-32U, symbol RF_Module:ESP32-WROOM-32U
- added C1: 100uF, Capacitor_Tantalum_SMD:CP_EIA-7343-43_Kemet-X, symbol Device:C_Polarized_Small
- added C5: 68uF, Capacitor_Tantalum_SMD:CP_EIA-3216-18_Kemet-A, symbol Device:C_Polarized_Small
- added U2: ESP32-WROOM-32D, RF_Module:ESP32-WROOM-32, symbol RF_Module:ESP32-WROOM-32D
- renumbered J2 to J1, J1 to J2
Connections:
- net IO33 is gone; now on net RTS: U3.11
- net +12V: now also C1.1
- net EN: now also U2.3 (EN)
- net E_EN: now also U2.28 (IO17)
- net GND: now also C1.2, C5.2, U2.1 (GND), U2.15 (GND), U2.38 (GND), U2.39 (GND)
- net IO0: now also U2.25 (IO0)
- net IO32: now also U2.8 (IO32)
- net RTS: now also U2.9 (IO33)
- net RXD0: now also U2.34 (RXD0/IO3)
- net RXG: now also U2.37 (IO23)
- net TXD0: now also U2.35 (TXD0/IO1)
- net TXG: now also U2.36 (IO22)
- net VCC: now also C5.1, U2.2 (VDD)
- net W_EN: now also U2.27 (IO16)
- net W_MOD: now also U2.31 (IO19)
- net W_RST: now also U2.30 (IO18)
- net BUSY: no longer names the net of J1.6, R3.2, U3.12, U3.8
Other:
- company: (none) -> Hyiger Designs
- title: (none) -> Celestron WiFi Adapter
